File: Hardware/OSSM_Main_PCB.brd (EAGLE design)
At the start: 128 x 51 mm, 11 parts, among them J1 PJ-037AH, U1 LOLIN32_PRODUCTION

Commit message: changes from initial PCB
Parts:
- moved J1 6.14 mm to (5.89, 33.1), turned to 180 degrees
Connections:
- net N$10: now also STEPPER.13; no longer STEPPER.11
- net N$8: now also STEPPER.11; no longer STEPPER.12
- net N$9: now also STEPPER.12; no longer STEPPER.13
Routing:
- net 24V: track 130.8 -> 119.0 mm
- net GND: track 268.6 -> 275.8 mm
- net N$10: track 19.5 -> 17.0 mm, vias 1 -> 0
- net N$8: track 20.6 -> 19.1 mm
- net N$9: track 19.1 -> 18.0 mm
Other:
- board text added: "+"
- board text added: "-"
- board text added: "24v"
- board text added: "5v"
