File: Hardware/PCB Files/OSSM Reference PCB V3/Power.kicad_sch (KiCad schematic)
At the start: 29 parts, among them J1 Screw_Terminal_01x02, J5 USB_C_Receptacle_USB2.0_16P, Q4 40P04, U1 LMR14006, U2 ME6211C33, U5 HUSB238

Commit message: Improved documentation and silkscreen
Parts:
- JP1: now not fitted
Other:
- company: (none) -> Research & Desire
- title: (none) -> OSSM!
Changed lines of the file:
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@@
 	(generator_version "8.0")
 	(paper "A4")
+	(title_block
+		(title "OSSM!")
+		(date "2024-08-21")
+		(rev "V3.0 Beta 1")
+		(company "Research & Desire")
+	)
 	(junction
 		(at 228.6 123.19)
@@
 		(in_bom no)
 		(on_board yes)
-		(dnp no)
+		(dnp yes)
 		(fields_autoplaced yes)
 		(property "Reference" "JP1"

Commit message: Last double check before ordering
Add Test points and Resistor Part numbers
Parts:
- C1: MPN C77020 -> C56392
- R14: MPN (none) -> C11702
- R18: MPN (none) -> C25077
- R2: MPN (none) -> C5126159
- R3: MPN (none) -> C60490
Changed lines of the file:
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@@
 			)
 		)
-		(property "MPN" ""
+		(property "MPN" "C25077"
 			(at 121.92 44.45 0)
 			(effects
@@
 			)
 		)
+		(property "MPN" "C11702"
+			(at 256.54 128.27 0)
+			(effects
+				(font
+					(size 1.27 1.27)
+				)
+				(hide yes)
+			)
+		)
 		(pin "2"
 		)
@@
 			)
 		)
+		(property "MPN" "C5126159"
+			(at 137.16 124.46 0)
+			(effects
+				(font
+					(size 1.27 1.27)
+				)
+				(hide yes)
+			)
+		)
 		(pin "1"
 		)
@@
 			)
 		)
+		(property "MPN" "C60490"
+			(at 137.16 133.35 0)
+			(effects
+				(font
+					(size 1.27 1.27)
+				)
+				(hide yes)
+			)
+		)
 		(pin "1"
 		)
@@
 			)
 		)
-		(property "Datasheet" "https://www.lcsc.com/product-detail/Multilayer-Ceramic-Capacitors-MLCC-SMD-SMT_Murata-Electronics-GRM155R71H104KE14D_C77020.html"
+		(property "Datasheet" "https://www.lcsc.com/datasheet/lcsc_datasheet_2304140030_FH--Guangdong-Fenghua-Advanced-Tech-0402B104K250NT_C56392.pdf"
 			(at 97.79 115.57 0)
 			(effects
@@
 			)
 		)
-		(property "MPN" "C77020"
+		(property "MPN" "C56392"
 			(at 97.79 115.57 0)
 			(effects
