File: Hardware/PCB Files/OSSM Reference PCB V3/mcu.kicad_sch (KiCad schematic)
At the start: 12 parts, among them J7 Conn_01x03, SW1 SW_Push, SW2 SW_Push, U7 ESP32-S3-WROOM-1

Commit message: Improved documentation and silkscreen
Parts:
- J7: now not fitted; now left out of the parts list
Other:
- company: (none) -> Research & Desire
- title: (none) -> OSSM!
Changed lines of the file:
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@@
 	(generator_version "8.0")
 	(paper "A4")
+	(title_block
+		(title "OSSM!")
+		(date "2024-08-21")
+		(rev "V3.0 Beta 1")
+		(company "Research & Desire")
+	)
 	(junction
 		(at 212.09 71.12)
@@
 		(unit 1)
 		(exclude_from_sim no)
-		(in_bom yes)
+		(in_bom no)
 		(on_board yes)
-		(dnp no)
+		(dnp yes)
 		(fields_autoplaced yes)
 		(property "Reference" "J7"

Commit message: Last double check before ordering
Add Test points and Resistor Part numbers
Parts:
- added TP1, TP2, TP3, TP4, TP5: TestPoint, TestPoint:TestPoint_Pad_1.0x1.0mm, symbol Connector:TestPoint
- C16, C8: MPN C77020 -> C56392
- R11, R12: MPN (none) -> C60490
- R8, R9: MPN (none) -> C11702
Connections:
- net at U7.17 (IO9): now also TP1.1
- net at U7.18 (IO10): now also TP2.1
- net at U7.19 (IO11): now also TP3.1
- net at U7.20 (IO12): now also TP4.1
- net at U7.21 (IO13): now also TP5.1
