File: Hardware/PCB Files/OSSM Reference PCB V3/motor.kicad_sch (KiCad schematic)
At the start: 18 parts, among them J2 Screw_Terminal_01x02, J4 Conn_01x04, J6 Conn_01x04, Q1 BC817, Q2 BC817, U3 INA219AIDCN, U4 SP3485EN

Commit message: Improved documentation and silkscreen
Parts:
- J4: now left out of the parts list
- J6: now fitted
Other:
- company: (none) -> Research & Desire
- title: (none) -> OSSM!
Changed lines of the file:
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@@
 	(generator_version "8.0")
 	(paper "A4")
+	(title_block
+		(title "OSSM!")
+		(date "2024-08-21")
+		(rev "V3.0 Beta 1")
+		(company "Research & Desire")
+	)
 	(junction
 		(at 93.98 55.88)
@@
 		(unit 1)
 		(exclude_from_sim no)
-		(in_bom yes)
+		(in_bom no)
 		(on_board yes)
 		(dnp no)
@@
 		)
 		(property "Description" "Generic connector, single row, 01x04, script generated (kicad-library-utils/schlib/autogen/connector/)"
-			(at 91.44 140.97 0)
-			(effects
-				(font
-					(size 1.27 1.27)
-				)
-				(hide yes)
-			)
-		)
-		(property "Sim.Type" ""
 			(at 91.44 140.97 0)
 			(effects
@@
 		(in_bom no)
 		(on_board yes)
-		(dnp yes)
+		(dnp no)
 		(fields_autoplaced yes)
 		(property "Reference" "J6"

Commit message: Last double check before ordering
Add Test points and Resistor Part numbers
Parts:
- C11: MPN C77020 -> C56392
- J6: now not fitted
- R22, R5: MPN (none) -> C25077
- R6, R7: MPN (none) -> C112291
Changed lines of the file:
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@@
+			)
+		)
+		(property "MPN" "C112291"
+			(at 46.99 146.05 0)
+			(effects
+				(font
+					(size 1.27 1.27)
+				)
+				(hide yes)
 			)
 		)
@@
 			)
 		)
+		(property "MPN" "C112291"
+			(at 67.31 158.75 0)
+			(effects
+				(font
+					(size 1.27 1.27)
+				)
+				(hide yes)
+			)
+		)
 		(pin "1"
 		)
@@
 			)
 		)
-		(property "MPN" ""
+		(property "MPN" "C25077"
 			(at 80.01 53.34 0)
 			(effects
@@
 			)
 		)
-		(property "Datasheet" "~"
+		(property "Datasheet" "https://www.lcsc.com/datasheet/lcsc_datasheet_2304140030_FH--Guangdong-Fenghua-Advanced-Tech-0402B104K250NT_C56392.pdf"
 			(at 59.69 39.37 0)
 			(effects
@@
 		(in_bom no)
 		(on_board yes)
-		(dnp no)
+		(dnp yes)
 		(fields_autoplaced yes)
 		(property "Reference" "J6"
@@
 			)
 		)
-		(property "Datasheet" "https://www.lcsc.com/product-detail/Multilayer-Ceramic-Capacitors-MLCC-SMD-SMT_Murata-Electronics-GRM155R71H104KE14D_C77020.html"
+		(property "Datasheet" "https://www.lcsc.com/datasheet/lcsc_datasheet_2304140030_FH--Guangdong-Fenghua-Advanced-Tech-0402B104K250NT_C56392.pdf"
 			(at 228.6 90.17 0)
 			(effects
@@
 			)
 		)
-		(property "MPN" "C77020"
+		(property "MPN" "C56392"
 			(at 228.6 90.17 0)
 			(effects
@@
 			)
 		)
-		(property "Datasheet" "~"
+		(property "Datasheet" "https://www.lcsc.com/datasheet/lcsc_datasheet_2304140030_FH--Guangdong-Fenghua-Advanced-Tech-0402B104K250NT_C56392.pdf"
 			(at 66.04 50.8 0)
 			(effects
@@
 			)
 		)
-		(property "MPN" ""
+		(property "MPN" "C25077"
 			(at 80.01 48.26 0)
 			(effects
