File: Hardware/PCB Files/OSSM Reference PCB V3/remote.kicad_sch (KiCad schematic)
At the start: 3 parts, among them J3 RJ45

Commit message: Improved documentation and silkscreen
Other:
- company: (none) -> Research & Desire
- title: (none) -> OSSM!
Changed lines of the file:
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@@
 	(generator_version "8.0")
 	(paper "A4")
+	(title_block
+		(title "OSSM!")
+		(date "2024-08-21")
+		(rev "V3.0 Beta 1")
+		(company "Research & Desire")
+	)
 	(junction
 		(at 143.51 93.98)

Commit message: Last double check before ordering
Add Test points and Resistor Part numbers
Parts:
- R10: MPN (none) -> C25792
- R13: MPN (none) -> C60490
Changed lines of the file:
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@@
+			)
+		)
+		(property "MPN" "C60490"
+			(at 152.4 104.14 0)
+			(effects
+				(font
+					(size 1.27 1.27)
+				)
+				(hide yes)
 			)
 		)
@@
 			(at 143.51 104.14 0)
 			(effects
+				(font
+					(size 1.27 1.27)
+				)
+				(hide yes)
+			)
+		)
+		(property "MPN" "C25792"
+			(at 143.51 104.14 0)
+			(effects
